Commit message: Simple Pick and Place Simulation

File: configured_urdf/urdf/arm_urdf.urdf (robot description, URDF)
Before this commit: robot arm_urdf, 10 links, 9 joints
Links:
- link base_link: geometry collision mesh filename=package://configured_urdf/meshes/base_link.STL; visual mesh filename=package://configured_urdf/meshes/base_link.STL
- link left_gripper: geometry collision mesh filename=package://configured_urdf/meshes/left_gripper.STL; visual mesh filename=package://configured_urdf/meshes/left_gripper.STL
- link link_1: geometry collision mesh filename=package://configured_urdf/meshes/link_1.STL; visual mesh filename=package://configured_urdf/meshes/link_1.STL
- link link_2: geometry collision mesh filename=package://configured_urdf/meshes/link_2.STL; visual mesh filename=package://configured_urdf/meshes/link_2.STL
- link link_3: geometry collision mesh filename=package://configured_urdf/meshes/link_3.STL; visual mesh filename=package://configured_urdf/meshes/link_3.STL
- link link_4: geometry collision mesh filename=package://configured_urdf/meshes/link_4.STL; visual mesh filename=package://configured_urdf/meshes/link_4.STL
- link link_5: geometry collision mesh filename=package://configured_urdf/meshes/link_5.STL; visual mesh filename=package://configured_urdf/meshes/link_5.STL
- link link_6: geometry collision mesh filename=package://configured_urdf/meshes/link_6.STL; visual mesh filename=package://configured_urdf/meshes/link_6.STL
- link right_gripper: geometry collision mesh filename=package://configured_urdf/meshes/right_gripper.STL; visual mesh filename=package://configured_urdf/meshes/right_gripper.STL

Commit message: World

File: configured_urdf/urdf/arm_urdf.urdf (robot description, URDF)
Before this commit: robot arm_urdf, 10 links, 9 joints
Joints:
- joint base_joint: origin xyz=0.0 0.0 0.17 rpy=0 0 0 -> xyz=0.0 0.0 1.205 rpy=0 0 0

Commit message: Maintenance Task Simulation

File: configured_urdf/urdf/arm_urdf.urdf (robot description, URDF)
Before this commit: robot arm_urdf, 10 links, 9 joints
Joints:
- joint base_joint: origin xyz=0.0 0.0 1.205 rpy=0 0 0 -> xyz=0.0 0.0 0.87 rpy=0 0 0

Commit message: Maintenance Task Simulation

File: configured_urdf/urdf/arm_urdf.urdf (robot description, URDF)
Before this commit: robot arm_urdf, 10 links, 9 joints
Joints:
- joint base_joint: origin xyz=0.0 0.0 0.87 rpy=0 0 0 -> xyz=0.0 0.0 1.2 rpy=0 0 0

File: maintenance_task_simulation/urdf/button.xacro (robot description, xacro)
@@ -23,4 +23,28 @@
       <origin xyz="1.431 0.18 1.05" rpy="1.5707 0.0 -1.5707"/>
     </joint>
+    <link name="number1">
+      <visual>
+        <geometry>
+          <mesh filename="package://maintenance_task_simulation/meshes/numbers/one.dae" scale="0.0006 0.0006 0.0006"/>
+        </geometry>
+      </visual>
+      <collision>
+        <geometry>
+          <mesh filename="package://maintenance_task_simulation/meshes/numbers/one.dae" scale="0.0006 0.0006 0.0006"/>
+        </geometry>
+      </collision>
+      <inertial>
+        <mass value="10" />
+        <inertia ixx="1.0" ixy="0.0" ixz="0.0" iyy="1.0" iyz="0.0" izz="1.0" />
+      </inertial>
+    </link>
+    <joint name="number1_joint" type="fixed">
+      <parent link="button1"/>
+      <child link="number1"/>
+      <origin xyz="0 0 0.07" rpy="0 0.0 0"/>
+    </joint>
+    <gazebo reference="number1">
+      <material>Gazebo/Black</material>
+    </gazebo>
     <link name="button2">
       <visual>
@@ -44,4 +68,28 @@
       <origin xyz="1.431 -0.18 1.05" rpy="1.5707 0.0 -1.5707"/>
     </joint>
+    <link name="number5">
+      <visual>
+        <geometry>
+          <mesh filename="package://maintenance_task_simulation/meshes/numbers/five.dae" scale="0.0006 0.0006 0.0006"/>
+        </geometry>
+      </visual>
+      <collision>
+        <geometry>
+          <mesh filename="package://maintenance_task_simulation/meshes/numbers/five.dae" scale="0.0006 0.0006 0.0006"/>
+        </geometry>
+      </collision>
+      <inertial>
+        <mass value="10" />
+        <inertia ixx="1.0" ixy="0.0" ixz="0.0" iyy="1.0" iyz="0.0" izz="1.0" />
+      </inertial>
+    </link>
+    <joint name="number5_joint" type="fixed">
+      <parent link="button2"/>
+      <child link="number5"/>
+      <origin xyz="0 0 0.07" rpy="0 0.0 0"/>
+    </joint>
+    <gazebo reference="number5">
+      <material>Gazebo/Black</material>
+    </gazebo>
     <link name="button3">
       <visual>
@@ -65,4 +113,28 @@
       <origin xyz="1.431 0.18 0.51" rpy="1.5707 0.0 -1.5707"/>
     </joint>
+    <link name="number8">
+      <visual>
+        <geometry>
+          <mesh filename="package://maintenance_task_simulation/meshes/numbers/eight.dae" scale="0.0006 0.0006 0.0006"/>
+        </geometry>
+      </visual>
+      <collision>
+        <geometry>
+          <mesh filename="package://maintenance_task_simulation/meshes/numbers/eight.dae" scale="0.0006 0.0006 0.0006"/>
+        </geometry>
+      </collision>
+      <inertial>
+        <mass value="10" />
+        <inertia ixx="1.0" ixy="0.0" ixz="0.0" iyy="1.0" iyz="0.0" izz="1.0" />
+      </inertial>
+    </link>
+    <joint name="number8_joint" type="fixed">
+      <parent link="button3"/>
+      <child link="number8"/>
+      <origin xyz="0 0 0.07" rpy="0 0.0 0"/>
+    </joint>
+    <gazebo reference="number8">
+      <material>Gazebo/Black</material>
+    </gazebo>
     <link name="button4">
       <visual>
@@ -86,4 +158,28 @@
       <origin xyz="1.431 -0.18 0.51" rpy="1.5707 0.0 -1.5707"/>
     </joint>
+    <link name="number3">
+      <visual>
+        <geometry>
+          <mesh filename="package://maintenance_task_simulation/meshes/numbers/three.dae" scale="0.0006 0.0006 0.0006"/>
+        </geometry>
+      </visual>
+      <collision>
+        <geometry>
+          <mesh filename="package://maintenance_task_simulation/meshes/numbers/three.dae" scale="0.0006 0.0006 0.0006"/>
+        </geometry>
+      </collision>
+      <inertial>
+        <mass value="10" />
+        <inertia ixx="1.0" ixy="0.0" ixz="0.0" iyy="1.0" iyz="0.0" izz="1.0" />
+      </inertial>
+    </link>
+    <joint name="number3_joint" type="fixed">
+      <parent link="button4"/>
+      <child link="number3"/>
+      <origin xyz="0 0 0.07" rpy="0 0.0 0"/>
+    </joint>
+    <gazebo reference="number3">
+      <material>Gazebo/Black</material>
+    </gazebo>
   </xacro:macro>
 </robot>
